Commit message: gripper fix test + simulation reset service

File: src/abb_irb120_description/urdf/gripper_macro.xacro (robot description, xacro)
@@ -83,5 +83,5 @@
         <origin xyz="0 0 0" rpy="0 0 0"/>
         <axis xyz="0 -1 0"/>
-        <limit lower="0.0" upper="0.01" effort="150" velocity="0.05"/>
+        <limit lower="-0.001" upper="0.011" effort="300" velocity="0.05"/>
         <dynamics damping="5.0" friction="0.5"/>
     </joint>
@@ -92,5 +92,5 @@
         <axis xyz="0 1 0"/>
         <mimic joint="${prefix}left_finger_joint" multiplier="1.0" offset="0.0"/>
-        <limit lower="0.0" upper="0.01" effort="150" velocity="0.05"/>
+        <limit lower="-0.001" upper="0.011" effort="300" velocity="0.05"/>
         <dynamics damping="5.0" friction="0.5"/>
     </joint>
